File: kicad/manette.kicad_pcb (KiCad board)
At the start: 2 copper layers, 127 x 101.6 mm, 31 parts, among them X1 SW_Push, Y1 SW_Push

Commit message: ajout d'un joystick achetable
Parts:
- added J1: THB001P, LibPerso:Joystick_THB001P, F.Cu at (206.5, 133.3)
- added R_B2: 100k, Resistor_THT:R_Axial_DIN0411_L9.9mm_D3.6mm_P15.24mm_Horizontal, F.Cu at (199.9, 147.1)
Connections:
- PUCE1 pad 1: 1 -> JOY_C_Y
- PUCE1 pad 2: 2 -> JOY_C_X
Routing:
- net JOY_C_A: track 0.00 -> 13.3 mm
- net 5V: track 187.3 -> 196.6 mm, vias 8 -> 12
